File: KiCAD/Carrier Board/melonHD.kicad_pcb (KiCad board)
At the start: 4 copper layers, 39 x 20 mm, 16 parts, among them J1 XUNPU HDMI-201, J4 USB_C_Receptacle, U1 ESD204DQAR-ES, U2 ESD204DQAR-ES, U3 ESD204DQAR-ES

Commit message: Update carrier board
Parts:
- J1: renamed from J4; value USB_C_Receptacle -> XUNPU TYPEC-324G-BCP24 or GCT USB4080-03-A
- J2: renamed from J1; value XUNPU HDMI-201 -> XUNPU HDMI-201 or Würth 685119136923
- renumbered TP5 to TP1, TP1 to TP2, TP2 to TP3, TP3 to TP5, U4 to U1, U1 to U2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
Routing:
- net GND: track 7.36 -> 6.79 mm, vias 127 -> 128
