File: KiCAD/Carrier Board/melonHD.kicad_sch (KiCad schematic)
At the start: 16 parts, among them J1 XUNPU HDMI-201, J4 USB_C_Receptacle, U1 ESD204DQAR-ES, U2 ESD204DQAR-ES, U3 ESD204DQAR-ES

Commit message: Update melonHD.kicad_sch
Other:
- note added: "NOTE: 3.3V output pin is for pinstrapping only. Do not connect an external load >50mA."
- note added: "PD VBUS Selection"
Changed lines of the file:
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@@
+		)
+	)
+	(text "NOTE: 3.3V output pin is \nfor pinstrapping only.\nDo not connect an external load >50mA."
+		(exclude_from_sim no)
+		(at 182.88 52.07 0)
+		(effects
+			(font
+				(size 1.27 1.27)
+				(thickness 0.254)
+				(bold yes)
+			)
+			(justify right)
+		)
+	)
+	(text "PD VBUS Selection"
+		(exclude_from_sim no)
+		(at 164.9378 62.6158 0)
+		(effects
+			(font
+				(size 1.27 1.27)
+				(thickness 0.254)
+				(bold yes)
+			)
+			(justify right)
 		)
 	)
@@
 		)
 	)
+	(polyline
+		(pts
+			(xy 193.2177 60.3333) (xy 193.2911 60.3333)
+		)
+		(stroke
+			(width 0)
+			(type default)
+		)
+	)
 	(wire
 		(pts
@@
 		)
 		(stroke
+			(width 0)
+			(type default)
+		)
+	)
+	(polyline
+		(pts
+			(xy 183.3862 51.6757) (xy 193.2177 60.3333)
+		)
+		(stroke

Commit message: Update carrier board
Parts:
- J1: renamed from J4; value USB_C_Receptacle -> GCT USB4080-03-A or XUNPU TYPEC-324G-BCP24
- J2: renamed from J1; value XUNPU HDMI-201 -> XUNPU HDMI-201 or Würth 685119136923
- renumbered TP5 to TP1, TP1 to TP2, TP2 to TP3, TP3 to TP5, U4 to U1, U1 to U2, U2 to U3, U3 to U4
Connections:
- net GND: now also J1.1 (SHIELD), J1.G1 (SHIELD), J1.G2 (SHIELD), J1.G3 (SHIELD), J1.G4 (SHIELD), J2.20 (GND), J2.21 (GND), J2.22 (GND), J2.23 (GND); no longer J1.S1 (SHIELD), J2.SH
Other:
- note added: "HPD Behavior: LOW (0V) - DP Alt Mode contract HIGH (3.3V) - Power-only contract"
- note added: "NOTE: 3.3V output pin is for pinstrapping / IO only. Do not connect an external load >50mA."
- note removed: "HPD Behavior: LOW (0V) - Power-only contract HIGH (3.3V) - DP Alt Mode contract"
- note removed: "NOTE: 3.3V output pin is for pinstrapping only. Do not connect an external load >50mA."

Commit message: Update schematic notes
Other:
- note added: "HPD Behavior: LOW (0V) - Power-only contract HIGH (3.3V) - DP Alt Mode contract"
- note removed: "HPD Behavior: LOW (0V) - DP Alt Mode contract HIGH (3.3V) - Power-only contract"
Changed lines of the file:
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@@
 		)
 	)
-	(text "HPD Behavior:\nLOW (0V) - DP Alt Mode contract\nHIGH (3.3V) - Power-only contract"
+	(text "HPD Behavior:\nLOW (0V) - Power-only contract\nHIGH (3.3V) - DP Alt Mode contract"
 		(exclude_from_sim no)
 		(at 200.66 106.68 0)

Commit message: Update module symbol
Parts:
- U1: footprint melonHD:melonHD_SMT -> SamacSys_Parts:lt6711a_smt
Changed lines of the file:
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@@
 			)
 		)
-		(property "Footprint" "melonHD:melonHD_SMT"
+		(property "Footprint" "SamacSys_Parts:lt6711a_smt"
 			(at 229.87 77.47 0)
 			(effects

Commit message: Update carrier board and fix 3D embed
Parts:
- U1: footprint SamacSys_Parts:lt6711a_smt -> melonhd_module:melonHD_SMT
Changed lines of the file:
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@@
 			)
 		)
-		(property "Footprint" "SamacSys_Parts:lt6711a_smt"
+		(property "Footprint" "melonhd_module:melonHD_SMT"
 			(at 229.87 77.47 0)
 			(effects
